File: hardware/usbXR.brd (EAGLE design)
At the start: 25.1 x 16.6 mm, 18 parts, among them SW1 BUTTON, U2 XC6206, U3 RFM70SMD_ONLY, U4 ATMEGA328P_TQFP, X1 USB-A-H, Y1 12MHz

Commit message: schematic in PNG
Parts:
- U3: value RFM70SMD_ONLY -> RFM70
Changed lines of the file:
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@@
 <attribute name="VALUE" x="19.685" y="6.223" size="1.27" layer="27" ratio="10" rot="R180"/>
 </element>
-<element name="U3" library="RFM70" package="RFM70_SMD" value="RFM70SMD_ONLY" x="24.892" y="3.81" smashed="yes" rot="MR90">
+<element name="U3" library="RFM70" package="RFM70_SMD" value="RFM70" x="24.892" y="3.81" smashed="yes" rot="MR90">
 <attribute name="NAME" x="6.858" y="15.494" size="0.8128" layer="26" font="vector" ratio="14" rot="MR0"/>
 <attribute name="VALUE" x="5.207" y="3.81" size="1.27" layer="28" rot="MR90"/>
