File: hardware/usbXR.sch (EAGLE design)
At the start: 18 parts, among them SW1 BUTTON, U2 XC6206, U3 RFM70SMD_ONLY, U4 ATMEGA328P_TQFP, X1 USB-A-H, Y1 12MHz

Commit message: schematic in PNG
Parts:
- U3: value RFM70SMD_ONLY -> RFM70
Changed lines of the file:
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@@
 <part name="GND11" library="supply1" deviceset="GND" device=""/>
 <part name="SUPPLY3" library="SparkFun-Aesthetics" deviceset="3.3V" device=""/>
-<part name="U3" library="RFM70" deviceset="RFM70" device="SMD_ONLY"/>
+<part name="U3" library="RFM70" deviceset="RFM70" device="SMD_ONLY" value="RFM70"/>
 <part name="U4" library="SparkFun-IC-Microcontroller" deviceset="ATMEGA328P_TQFP" device="" value="ATMEGA328P_TQFP"/>
 </parts>
